File: EagleFirstHW/projects/attiny85_transistor/attiny85_transistor.brd (EAGLE design)
At the start: 100 x 80 mm, 19 parts, among them Q1 BSH103

Commit message: adding marquee
Routing:
- net 5V: track 285.0 -> 273.2 mm
- net N$8: track 0.00 -> 4.52 mm
- net N$7: track 0.00 -> 4.52 mm
- net N$1: track 0.00 -> 4.52 mm
- net N$9: track 0.71 -> 3.97 mm
- net N$10: track 0.00 -> 3.25 mm
Changed lines of the file:
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@@
 <contactref element="R4" pad="1"/>
 <contactref element="LED1" pad="A"/>
-<wire x1="91.44" y1="57.47" x2="91.44" y2="52.947" width="0" layer="19" extent="1-1"/>
+<wire x1="91.44" y1="57.47" x2="91.44" y2="52.947" width="0.4064" layer="1"/>
 </signal>
 <signal name="N$7">
 <contactref element="R5" pad="1"/>
 <contactref element="LED2" pad="A"/>
-<wire x1="83.82" y1="52.947" x2="83.82" y2="57.47" width="0" layer="19" extent="1-1"/>
+<wire x1="83.82" y1="57.47" x2="83.82" y2="52.947" width="0.4064" layer="1"/>
 </signal>
 <signal name="N$8">
 <contactref element="R6" pad="1"/>
 <contactref element="LED3" pad="A"/>
-<wire x1="76.2" y1="52.947" x2="76.2" y2="57.47" width="0" layer="19" extent="1-1"/>
+<wire x1="76.2" y1="57.47" x2="76.2" y2="52.947" width="0.4064" layer="1"/>
 </signal>
 <signal name="N$9">
@@
 <contactref element="LED4" pad="A"/>
 <wire x1="71.12" y1="54.93" x2="71.12" y2="54.217" width="0.4064" layer="1"/>
-<wire x1="71.12" y1="54.93" x2="71.12" y2="57.47" width="0" layer="19" extent="1-1"/>
+<wire x1="71.12" y1="57.47" x2="71.12" y2="54.217" width="0.4064" layer="1"/>
 </signal>
 <signal name="N$10">
 <contactref element="R8" pad="1"/>
 <contactref element="LED5" pad="A"/>
-<wire x1="62.23" y1="54.217" x2="62.23" y2="57.47" width="0" layer="19" extent="1-1"/>
+<wire x1="62.23" y1="57.47" x2="62.23" y2="54.217" width="0.4064" layer="1"/>
 </signal>
 <signal name="N$4">
@@
 <wire x1="33.02" y1="53.34" x2="41.54" y2="53.34" width="0.4064" layer="1"/>
 <wire x1="41.54" y1="53.34" x2="44.45" y2="50.43" width="0.4064" layer="1"/>
-<wire x1="45.4655375" y1="50.0332" x2="46.0532" y2="49.4455375" width="0.4064" layer="1"/>
-<wire x1="44.2305375" y1="35.1918" x2="42.8118" y2="35.1918" width="0.4064" layer="1"/>
-<wire x1="42.8118" y1="35.1918" x2="41.91" y2="34.29" width="0.4064" layer="1"/>
 <wire x1="44.45" y1="50.43" x2="44.8468" y2="50.0332" width="0.4064" layer="1"/>
-<wire x1="44.8468" y1="50.0332" x2="45.4655375" y2="50.0332" width="0.4064" layer="1"/>
-<wire x1="46.0532" y1="49.4455375" x2="46.0532" y2="37.0144625" width="0.4064" layer="1"/>
-<wire x1="46.0532" y1="37.0144625" x2="44.52436875" y2="35.48563125" width="0.4064" layer="1"/>
-<wire x1="44.52436875" y1="35.48563125" x2="44.2305375" y2="35.1918" width="0.4064" layer="1"/>
-<wire x1="41.91" y1="34.29" x2="41.545" y2="34.29" width="0.4064" layer="1"/>
-<wire x1="57.29" y1="19.05" x2="44.52436875" y2="31.81563125" width="0.4064" layer="1"/>
-<wire x1="44.52436875" y1="31.81563125" x2="44.52436875" y2="35.48563125" width="0.4064" layer="1"/>
 <wire x1="74.93" y1="41.91" x2="74.93" y2="46.62" width="0.4064" layer="1"/>
 <wire x1="62.23" y1="59.37" x2="61.8332" y2="58.9732" width="0.4064" layer="1"/>
 <wire x1="61.8332" y1="58.9732" x2="61.3144625" y2="58.9732" width="0.4064" layer="1"/>
-<wire x1="61.3144625" y1="58.9732" x2="60.7268" y2="58.3855375" width="0.4064" layer="1"/>
 <wire x1="70.2044625" y1="58.9732" x2="72.0355375" y2="58.9732" width="0.4064" layer="1"/>
-<wire x1="45.8259375" y1="50.43" x2="44.45" y2="50.43" width="0.4064" layer="1"/>
-<wire x1="49.1618" y1="47.0941375" x2="45.8259375" y2="50.43" width="0.4064" layer="1"/>
-<wire x1="49.1618" y1="42.12665" x2="49.1618" y2="47.0941375" width="0.4064" layer="1"/>
-<wire x1="45.7836" y1="38.74845" x2="49.1618" y2="42.12665" width="0.4064" layer="1"/>
-<wire x1="76.6085375" y1="54.4002" x2="92.27645625" y2="54.4002" width="0.4064" layer="1"/>
-<wire x1="72.0355375" y1="58.9732" x2="76.6085375" y2="54.4002" width="0.4064" layer="1"/>
-<wire x1="66.9014625" y1="55.6702" x2="70.2044625" y2="58.9732" width="0.4064" layer="1"/>
-<wire x1="60.7268" y1="58.3855375" x2="60.7268" y2="55.6702" width="0.4064" layer="1"/>
-<wire x1="60.7268" y1="55.6702" x2="66.9014625" y2="55.6702" width="0.4064" layer="1"/>
-<wire x1="95.3896" y1="34.7972625" x2="77.9391375" y2="17.3468" width="0.4064" layer="1"/>
-<wire x1="77.9391375" y1="17.3468" x2="60.1744625" y2="17.3468" width="0.4064" layer="1"/>
-<wire x1="60.1744625" y1="17.3468" x2="45.7836" y2="31.7376625" width="0.4064" layer="1"/>
-<wire x1="45.7836" y1="31.7376625" x2="45.7836" y2="38.74845" width="0.4064" layer="1"/>
-<wire x1="92.27645625" y1="54.4002" x2="95.3896" y2="51.28705625" width="0.4064" layer="1"/>
-<wire x1="95.3896" y1="51.28705625" x2="95.3896" y2="34.7972625" width="0.4064" layer="1"/>
+<wire x1="44.8468" y1="50.0332" x2="45.4655375" y2="50.0332" width="0.4064" layer="1"/>
+<wire x1="45.4655375" y1="50.0332" x2="46.99" y2="48.5087375" width="0.4064" layer="1"/>
+<wire x1="46.99" y1="37.2661125" x2="45.7836" y2="36.0597125" width="0.4064" layer="1"/>
+<wire x1="45.7836" y1="34.3536" x2="45.72" y2="34.29" width="0.4064" layer="1"/>
+<wire x1="45.7836" y1="36.0597125" x2="45.7836" y2="34.3536" width="0.4064" layer="1"/>
+<wire x1="46.99" y1="48.5087375" x2="46.99" y2="37.2661125" width="0.4064" layer="1"/>
+<wire x1="45.72" y1="34.29" x2="41.545" y2="34.29" width="0.4064" layer="1"/>
+<wire x1="45.7836" y1="34.3536" x2="45.7836" y2="26.6064" width="0.4064" layer="1"/>
+<wire x1="45.7836" y1="26.6064" x2="53.34" y2="19.05" width="0.4064" layer="1"/>
+<wire x1="53.34" y1="19.05" x2="57.29" y2="19.05" width="0.4064" layer="1"/>
+<wire x1="62.23" y1="59.37" x2="62.23" y2="62.23" width="0.4064" layer="1"/>
+<wire x1="62.23" y1="62.23" x2="92.71" y2="62.23" width="0.4064" layer="1"/>
+<wire x1="92.71" y1="62.23" x2="97.79" y2="57.15" width="0.4064" layer="1"/>
+<wire x1="97.79" y1="57.15" x2="97.79" y2="25.4" width="0.4064" layer="1"/>
+<wire x1="97.79" y1="25.4" x2="85.09" y2="12.7" width="0.4064" layer="1"/>
+<wire x1="85.09" y1="12.7" x2="53.34" y2="12.7" width="0.4064" layer="1"/>
+<wire x1="53.34" y1="12.7" x2="53.34" y2="19.05" width="0.4064" layer="1"/>
+<wire x1="71.12" y1="59.37" x2="70.2044625" y2="58.9732" width="0" layer="19" extent="1-1"/>
 </signal>
 </signals>
